Commit message: Add proper collision files for the base

File: tiago_pro_head_description/urdf/head_base.urdf.xacro (robot description, xacro)
@@ -28,5 +28,5 @@
         <geometry>
             <mesh
-            filename="package://tiago_pro_head_description/meshes/base_link.STL" />
+            filename="package://tiago_pro_head_description/meshes/base_link_collision.stl" />
         </geometry>
         </collision>
@@ -52,5 +52,5 @@
             <origin xyz="0 0 0" rpy="0 0 0" />
             <geometry>
-                <mesh filename="package://tiago_pro_head_description/meshes/head_base_link.STL" />
+                <mesh filename="package://tiago_pro_head_description/meshes/head_base_link_collision.STL" />
             </geometry>
         </collision>

Commit message: Update pm2

File: tiago_pro_head_description/urdf/head_base.urdf.xacro (robot description, xacro)
@@ -15,4 +15,11 @@
     <xacro:macro name="tiago_pro_head_base">
         <link name="base_link">
+        <inertial>
+            <origin xyz="0.00110975357790618 -8.60892376169405E-05 0.0747909538589444" rpy="0 0 0" />
+            <mass value="1.29631752086684" />
+            <inertia ixx="0.00493590257336928" ixy="-5.75640744380783E-05" ixz="0.000268460515456378"
+                iyy="0.00874689522512829" iyz="1.68556095053599E-05"
+                izz="0.0110057824631146" />
+        </inertial>
         <visual>
             <origin xyz="0 0 0" rpy="0 0 0" />
