Commit message: Align with tiago_pro fix on the origins of the base links for the head

File: tiago_pro_head_description/urdf/head.urdf.xacro (robot description, xacro)
@@ -29,27 +29,29 @@
     <!-- Head Link 1-->
     <link name="${name}_1_link">
-    <inertial>
-        <origin xyz="0.0016768 3.1033E-05 0.081737" rpy="0 0 0" />
-        <mass value="0.22677" />
-        <inertia ixx="0.00056619" ixy="3.0482E-07" ixz="6.7491E-05" iyy="0.00040222" iyz="-5.9322E-07" izz="0.00039176" />
-    </inertial>
-    <visual>
+      <inertial>
+        <origin xyz="-0.0037459 -4.6685E-05 0.1055" rpy="0 0 0" />
+        <mass value="0.15566" />
+        <inertia ixx="0.0005208" ixy="3.0453E-07" ixz="-6.1005E-05"
+          iyy="0.00035021" iyz="5.8627E-07"
+          izz="0.00033341" />
+      </inertial>
+      <visual>
         <origin xyz="0 0 0" rpy="0 0 0" />
         <geometry>
-        <mesh filename="package://tiago_pro_head_description/meshes/head_1_link.stl" />
+          <mesh filename="package://tiago_pro_head_description/meshes/head_1_link.stl" />
         </geometry>
         <material name="">
           <color rgba="0.29804 0.29804 0.29804 1" />
         </material>
-    </visual>
-    <collision>
+      </visual>
+      <collision>
         <origin xyz="0 0 0" rpy="0 0 0" />
         <geometry>
-        <mesh filename="package://tiago_pro_head_description/meshes/head_1_link_collision.stl" />
+          <mesh filename="package://tiago_pro_head_description/meshes/head_1_link_collision.stl" />
         </geometry>
-    </collision>
+      </collision>
     </link>
     <joint name="${name}_1_joint" type="revolute">
-      <origin xyz="0 0 0" rpy="0 0 3.14" />
+      <origin xyz="0 0 0" rpy="0 0 0" />
       <parent link="${parent}" />
       <child link="head_1_link" />
@@ -62,7 +64,9 @@
     <link name="${name}_2_link">
       <inertial>
-        <origin xyz="-0.0087157 0.11401 -0.00024206" rpy="0 0 0" />
-        <mass value="0.84465" />
-        <inertia ixx="0.006226" ixy="-0.00055126" ixz="-7.2157E-06" iyy="0.0050209" iyz="-1.0342E-05" izz="0.002495" />
+        <origin xyz="-0.00875103486217405 0.114127350051331 -0.000389070804431699"  rpy="0 0 0" />
+        <mass value="0.846359357446667" />
+        <inertia ixx="0.00623850186261437" ixy="-0.000550112126953165" ixz="-9.403405403969E-06"
+          iyy="0.0050320204467172" iyz="-5.68886635279132E-06"
+          izz="0.0024981099013485" />
       </inertial>
       <visual>
@@ -82,6 +86,6 @@
       </collision>
     </link>
-    <joint name="${name}_2_joint" type="revolute">
-      <origin xyz="-0.0425 0 0.1011" rpy="1.5708 0 0" />
+    <joint name="head_2_joint" type="revolute">
+      <origin xyz="0.0425 0 0.10585" rpy="1.5708 0 -3.1416" />
       <parent link="${name}_1_link" />
       <child link="${name}_2_link" />
@@ -115,5 +119,5 @@
     <!-- Head camera:Intel D435 -->
     <xacro:sensor_d435 parent="${name}_2_link" name="${name}_front_camera" topics_ns="${name}_front_camera" use_nominal_extrinsics="${use_sim_time}">
-      <origin xyz="-0.0415999999999995 0.1555 0" rpy="1.5707963267949 0 3.14159265358979" />
+      <origin xyz="-0.0416 0.1555 0" rpy="1.5708 0 3.1416" />
     </xacro:sensor_d435>
   </xacro:macro>

Commit message: Rotate sellion link

File: tiago_pro_head_description/urdf/head.urdf.xacro (robot description, xacro)
@@ -128,5 +128,5 @@
   <link name="sellion_link"/>
   <joint name="sellion_joint" type="fixed">
-    <origin xyz="0.04 0.09205 0" rpy="${-90 * deg_to_rad} 0 0"/>
+    <origin xyz="-0.04 0.09205 0" rpy="${-90 * deg_to_rad} ${180 * deg_to_rad} 0"/>
     <child link="sellion_link" />
     <parent link="head_2_link"/>

Commit message: Add libgazebo_ros_video plugin to TIAGo Pro Head

File: tiago_pro_head_description/urdf/head.urdf.xacro (robot description, xacro)
@@ -95,5 +95,26 @@
       <safety_controller k_position="20" k_velocity="20" soft_lower_limit="${head_2_lower_limit + head_eps}" soft_upper_limit="${head_2_upper_limit - head_eps}" />
     </joint>
-    <link name="${name}_screen_link"/>
+    <link name="${name}_screen_link">
+      <visual>
+        <origin rpy="${90.0 * deg_to_rad} 0 ${-90.0 * deg_to_rad}" xyz="-0.105 0 0"/>
+        <geometry>
+          <box size="0.17282 0.10824 0.005"/>
+        </geometry>
+      </visual>
+    </link>
+    <gazebo reference="${name}_screen_link">
+      <visual>
+        <plugin name="${name}_video_stream" filename="libgazebo_ros_video.so">
+          <ros>
+            <!-- Add a namespace -->
+            <namespace></namespace>
+            <!-- remap image subscribe topic -->
+            <remapping>~/image_raw:=robot_face/image_raw</remapping>
+          </ros>
+          <height>480</height>
+          <width>640</width>
+        </plugin>
+      </visual>
+    </gazebo>
     <joint name="${name}_screen_joint" type="fixed">
       <parent link="${name}_2_link" />

Commit message: Increase the safety factor due to the cable getting compressed at joint limits

File: tiago_pro_head_description/urdf/head.urdf.xacro (robot description, xacro)
@@ -25,5 +25,5 @@
   <xacro:property name="head_2_lower_limit" value="-1.0472"/>
   <xacro:property name="head_2_upper_limit" value="0.34907"/>
-  <xacro:property name="head_eps" value="${0.07}" />
+  <xacro:property name="head_eps" value="${0.15}" />
   <xacro:macro name="tiago_pro_head" params="name parent camera_model use_sim_time:=^|false">
     <!-- Head Link 1-->

Commit message: Add Realsense D455 to tiago pro head

File: tiago_pro_head_description/urdf/head.urdf.xacro (robot description, xacro)
@@ -15,4 +15,5 @@
   <!--File includes-->
   <xacro:include filename="$(find realsense2_description)/urdf/_d435.urdf.xacro" />
+  <xacro:include filename="$(find realsense2_description)/urdf/_d455.urdf.xacro" />
   <!-- Tools -->
   <xacro:include filename="$(find pal_urdf_utils)/urdf/deg_to_rad.urdf.xacro" />
@@ -70,4 +71,13 @@
           izz="0.00627" />
       </inertial>
+      <visual>
+        <origin xyz="0 0 0" rpy="0 0 0" />
+        <geometry>
+          <mesh filename="package://tiago_pro_head_description/meshes/${camera_model}_cover_link.stl" />
+        </geometry>
+        <material name="">
+          <color rgba="1 1 1 1" />
+        </material>
+      </visual>
       <visual>
         <origin xyz="0 0 0" rpy="0 0 0" />
@@ -148,4 +158,10 @@
       </xacro:sensor_d435>
     </xacro:if>
+    <!-- Head camera:Intel D455 -->
+    <xacro:if value="${camera_model == 'realsense-d455'}">
+      <xacro:sensor_d455 parent="${name}_2_link" name="${name}_front_camera" topics_ns="${name}_front_camera" use_nominal_extrinsics="${use_sim_time}">
+        <origin xyz="0.040453 -0.1565 0" rpy="1.5708 0 0" />
+      </xacro:sensor_d455>
+    </xacro:if>
   </xacro:macro>
   <!-- EYE FRAMES -->

Commit message: Put back old eps because this should be fixed for heads after the first one

File: tiago_pro_head_description/urdf/head.urdf.xacro (robot description, xacro)
@@ -26,5 +26,5 @@
   <xacro:property name="head_2_lower_limit" value="-1.0472"/>
   <xacro:property name="head_2_upper_limit" value="0.34907"/>
-  <xacro:property name="head_eps" value="${0.15}" />
+  <xacro:property name="head_eps" value="${0.07}" />
   <xacro:macro name="tiago_pro_head" params="name parent camera_model use_sim_time:=^|false">
     <!-- Head Link 1-->

Commit message: new frame for wbc addedd

File: tiago_pro_head_description/urdf/head.urdf.xacro (robot description, xacro)
@@ -184,3 +184,9 @@
     <parent link="sellion_link"/>
   </joint>
+  <link name="head_front_camera_color_eye_frame"/>
+  <joint name="color_eye_joint" type="fixed">
+    <origin xyz="-0.000 -0.059 -0.000" rpy="-1.566 0.002 -1.568"/>
+    <child link="head_front_camera_color_eye_frame" />
+    <parent link="head_front_camera_link"/>
+  </joint>
 </robot>

Commit message: adding depth frame for calibration

File: tiago_pro_head_description/urdf/head.urdf.xacro (robot description, xacro)
@@ -190,3 +190,9 @@
     <parent link="head_front_camera_link"/>
   </joint>
+  <link name="head_front_camera_depth_eye_frame"/>
+  <joint name="depth_eye_joint" type="fixed">
+    <origin xyz="0.000 0.000 0.000" rpy="-1.571 0.000 -1.571"/>
+    <child link="head_front_camera_depth_eye_frame" />
+    <parent link="head_front_camera_link"/>
+  </joint>
 </robot>

Commit message: Unifying frames

File: tiago_pro_head_description/urdf/head.urdf.xacro (robot description, xacro)
@@ -186,13 +186,7 @@
   <link name="head_front_camera_color_eye_frame"/>
   <joint name="color_eye_joint" type="fixed">
-    <origin xyz="-0.000 -0.059 -0.000" rpy="-1.566 0.002 -1.568"/>
+    <origin xyz="0.000 0.000 0.000" rpy="-1.571 0.000 -1.571"/>
     <child link="head_front_camera_color_eye_frame" />
     <parent link="head_front_camera_link"/>
   </joint>
-  <link name="head_front_camera_depth_eye_frame"/>
-  <joint name="depth_eye_joint" type="fixed">
-    <origin xyz="0.000 0.000 0.000" rpy="-1.571 0.000 -1.571"/>
-    <child link="head_front_camera_depth_eye_frame" />
-    <parent link="head_front_camera_link"/>
-  </joint>
 </robot>

Commit message: fix the parameter name to world_name and not world

File: tiago_pro_head_description/urdf/head.urdf.xacro (robot description, xacro)
@@ -167,5 +167,5 @@
     </xacro:if>
   </xacro:macro>
-  <xacro:macro name="tiago_pro_head_mj" params="mj_control world">
+  <xacro:macro name="tiago_pro_head_mj" params="mj_control world_name">
     <xacro:include filename="$(find tiago_pro_head_description)/mujoco/mj_tags.xacro" />
     <xacro:include filename="$(find pal_mujoco_scenes)/scenes/${world_name}.xacro" />

Commit message: Update head.urdf.xacro

File: tiago_pro_head_description/urdf/head.urdf.xacro (robot description, xacro)
@@ -155,4 +155,10 @@
     </gazebo>
     <!-- Cameras-->
+    <!-- Head camera:Intel D435i -->
+    <xacro:if value="${camera_model == 'realsense-d435i'}">
+      <xacro:realsense_d435i parent="${name}_2_link" name="${name}_front_camera" use_nominal_extrinsics="${use_sim_time}">
+        <origin xyz="0.0416 -0.1555 0" rpy="1.5708 0 0" />
+      </xacro:realsense_d435i>
+    </xacro:if>
     <!-- Head camera:Intel D435 -->
     <xacro:if value="${camera_model == 'realsense-d435'}">
