Commit message: create a xacro file with joint properties

File: tiago_pro_head_description/mujoco/mj_tags.xacro (robot description, xacro)
@@ -1,8 +1,9 @@
 <?xml version="1.0"?>
-<robot xmlns:xacro="http://ros.org/wiki/xacro" name="tiago_pro_head">
-    <xacro:macro name="mj_head_actuators">
+<robot xmlns:xacro="http://ros.org/wiki/xacro">
+    <xacro:macro name="mj_head_actuators" params="mj_control">
+        <xacro:include filename="$(find tiago_pro_head_description)/urdf/head_limits.xacro" />
         <xacro:if value="${mj_control == 'position'}">
-            <position name="head_1_joint_position" joint="head_1_joint" ctrlrange="-1.309 1.309" kp="2000" />
-            <position name="head_2_joint_position" joint="head_2_joint" ctrlrange="-1.0472 0.34907" kp="2000"/>
+            <position name="head_1_joint_position" joint="head_1_joint" ctrlrange="${head_1_lower_limit} ${head_1_upper_limit}" kp="2000" />
+            <position name="head_2_joint_position" joint="head_2_joint" ctrlrange="${head_2_lower_limit} ${head_2_upper_limit}" kp="2000"/>
         </xacro:if>
         <xacro:if value="${mj_control == 'motor'}">

File: tiago_pro_head_description/urdf/head.urdf.xacro (robot description, xacro)
@@ -14,20 +14,12 @@
 <robot xmlns:xacro="http://ros.org/wiki/xacro">
   <xacro:macro name="tiago_pro_head" params="name parent camera_model use_sim_time:=^|false">
-  <!--File includes-->
-  <xacro:include filename="$(find pal_urdf_utils)/urdf/camera/realsense_d435.urdf.xacro" />
-  <xacro:include filename="$(find pal_urdf_utils)/urdf/camera/realsense_d435i.urdf.xacro" />
-  <xacro:include filename="$(find pal_urdf_utils)/urdf/camera/realsense_d455.urdf.xacro" />
-  <!-- Tools -->
-  <xacro:include filename="$(find pal_urdf_utils)/urdf/deg_to_rad.urdf.xacro" />
-  <!--Constant parameters-->
-  <xacro:property name="head_friction" value="1.0" />
-  <xacro:property name="head_damping" value="0.5" />
-  <xacro:property name="head_max_vel" value="3.0" />
-  <xacro:property name="head_1_lower_limit" value="-1.309"/>
-  <xacro:property name="head_1_upper_limit" value="1.309"/>
-  <xacro:property name="head_2_lower_limit" value="-1.0472"/>
-  <xacro:property name="head_2_upper_limit" value="0.34907"/>
-  <xacro:property name="head_eps" value="${0.07}" />
-  <xacro:macro name="tiago_pro_head" params="name parent camera_model use_sim_time:=^|false">
+    <!--File includes-->
+    <xacro:include filename="$(find pal_urdf_utils)/urdf/camera/realsense_d435.urdf.xacro" />
+    <xacro:include filename="$(find pal_urdf_utils)/urdf/camera/realsense_d435i.urdf.xacro" />
+    <xacro:include filename="$(find pal_urdf_utils)/urdf/camera/realsense_d455.urdf.xacro" />
+     <!-- Tools -->
+    <xacro:property name="head_eps" value="${0.07}" />
+    <xacro:include filename="$(find pal_urdf_utils)/urdf/deg_to_rad.urdf.xacro" />
+    <xacro:include filename="$(find tiago_pro_head_description)/urdf/head_limits.xacro" />
     <!-- Head Link 1-->
     <link name="${name}_1_link">
@@ -60,5 +52,5 @@
       <child link="head_1_link" />
       <axis xyz="0 0 1" />
-      <limit lower="${head_1_lower_limit}" upper="${head_1_upper_limit}" effort="5.197" velocity="${head_max_vel}" />
+      <limit lower="${head_1_lower_limit}" upper="${head_1_upper_limit}" effort="${head_1_max_effort}" velocity="${head_max_vel}" />
       <dynamics damping="${head_damping}" friction="${head_friction}"/>
       <safety_controller k_position="20" k_velocity="20" soft_lower_limit="${head_1_lower_limit + head_eps}" soft_upper_limit="${head_1_upper_limit - head_eps}" />
@@ -103,5 +95,5 @@
       <child link="${name}_2_link" />
       <axis xyz="0 0 -1" />
-      <limit lower="${head_2_lower_limit}" upper="${head_2_upper_limit}" effort="2.77" velocity="${head_max_vel}" />
+      <limit lower="${head_2_lower_limit}" upper="${head_2_upper_limit}" effort="${head_2_max_effort}" velocity="${head_max_vel}" />
       <dynamics damping="${head_damping}" friction="${head_friction}"/>
       <safety_controller k_position="20" k_velocity="20" soft_lower_limit="${head_2_lower_limit + head_eps}" soft_upper_limit="${head_2_upper_limit - head_eps}" />
