Commit message: Add gazebo ignition for TIAGo Pro Head

File: tiago_pro_head_description/ros2_control/ros2_control.urdf.xacro (robot description, xacro)
@@ -17,22 +17,31 @@
     <xacro:unless value="$(arg use_sim_time)">
       <ros2_control name="ros2_control_tiago_pro_head_system" type="system">
-        <hardware>
-          <plugin>robot_control/RobotControl</plugin>
-        </hardware>
+          <hardware>
+            <xacro:if value="${use_sim_time}">
+              <xacro:if value="${gazebo_version == 'classic'}">
+                <plugin>gazebo_ros2_control/GazeboSystem</plugin>
+              </xacro:if>
+              <xacro:if value="${gazebo_version == 'gazebo'}">
+                <plugin>gz_ros2_control/GazeboSimSystem</plugin>
+              </xacro:if>
+            </xacro:if>
+            <xacro:unless value="${use_sim_time}">
+              <plugin>robot_control/RobotControl</plugin>
+            </xacro:unless>
+          </hardware>
         <xacro:ros2_control_head />
       </ros2_control>
     </xacro:unless>
-    <xacro:if value="$(arg use_sim_time)">
-      <gazebo>
-        <plugin filename="libgazebo_ros2_control.so" name="gazebo_ros2_control">
-          <parameters>$(find tiago_pro_head_description)/ros2_control/gazebo_controller_manager_cfg.yaml</parameters>
-        </plugin>
-      </gazebo>
-      <ros2_control name="ros2_control_head_gazebo_system" type="system">
-        <hardware>
-          <plugin>gazebo_ros2_control/GazeboSystem</plugin>
-        </hardware>
-        <xacro:ros2_control_head />
-      </ros2_control>
+    <xacro:if value="${gazebo_version == 'classic'}">
+      <plugin filename="libgazebo_ros2_control.so" name="gazebo_ros2_control">
+        <parameters>$(find tiago_pro_head_description)/ros2_control/gazebo_controller_manager_cfg.yaml</parameters>
+      </plugin>
+    </xacro:if>
+    <xacro:if value="${gazebo_version == 'gazebo'}">
+      <plugin filename="gz_ros2_control-system" name="gz_ros2_control::GazeboSimROS2ControlPlugin">
+        <robot_param>robot_description</robot_param>
+        <robot_param_node>robot_state_publisher</robot_param_node>
+        <parameters>$(find tiago_pro_head_description)/ros2_control/gazebo_controller_manager_cfg.yaml</parameters>
+      </plugin>
     </xacro:if>
   </xacro:macro>

File: tiago_pro_head_description/urdf/head.urdf.xacro (robot description, xacro)
@@ -116,18 +116,20 @@
       </visual>
     </link>
-    <gazebo reference="${name}_screen_link">
-      <visual>
-        <plugin name="${name}_video_stream" filename="libgazebo_ros_video.so">
-          <ros>
-            <!-- Add a namespace -->
-            <namespace></namespace>
-            <!-- remap image subscribe topic -->
-            <remapping>~/image_raw:=robot_face/image_raw</remapping>
-          </ros>
-          <height>480</height>
-          <width>640</width>
-        </plugin>
-      </visual>
-    </gazebo>
+    <xacro:if value="${gazebo_version == 'classic'}">
+      <gazebo reference="${name}_screen_link">
+        <visual>
+          <plugin name="${name}_video_stream" filename="libgazebo_ros_video.so">
+            <ros>
+              <!-- Add a namespace -->
+              <namespace></namespace>
+              <!-- remap image subscribe topic -->
+              <remapping>~/image_raw:=robot_face/image_raw</remapping>
+            </ros>
+            <height>480</height>
+            <width>640</width>
+          </plugin>
+        </visual>
+      </gazebo>
+    </xacro:if>
     <joint name="${name}_screen_joint" type="fixed">
       <parent link="${name}_2_link" />

Commit message: add missing sim_type parameter

File: tiago_pro_head_description/ros2_control/ros2_control.urdf.xacro (robot description, xacro)
@@ -13,5 +13,5 @@
  -->
 <robot xmlns:xacro="http://ros.org/wiki/xacro" name="tiago_pro_head" >
-  <xacro:macro name="tiago_pro_head_ros2_control" params="use_sim_time:=^|false">
+  <xacro:macro name="tiago_pro_head_ros2_control" params="use_sim_time:=^|false sim_type:=^|gazebo">
     <xacro:include filename="$(find tiago_pro_head_description)/urdf/head.ros2_control.xacro" />
     <ros2_control name="ros2_control_tiago_pro_head_system" type="system">
