Commit message: Add condition for cameras in urdf

File: tiago_pro_head_description/robots/tiago_pro_head.urdf.xacro (robot description, xacro)
@@ -14,6 +14,8 @@
 <robot xmlns:xacro="http://ros.org/wiki/xacro" name="tiago_pro_head">
   <xacro:include filename="$(find tiago_pro_head_description)/urdf/head.urdf.xacro" />
+  <xacro:arg name="camera_model" default="realsense-d435"/>
   <xacro:arg name="use_sim_time" default="false"/>
   <xacro:arg name="is_public_sim" default="false"/>
+  <xacro:property name="camera_model" value="$(arg camera_model)" />
   <xacro:property name="use_sim_time" value="$(arg use_sim_time)" />
   <xacro:property name="is_public_sim" value="$(arg is_public_sim)" />
@@ -23,4 +25,4 @@
   <xacro:include filename="$(find tiago_pro_head_description)/urdf/head_base.urdf.xacro" />
   <xacro:tiago_pro_head_base/>
-  <xacro:tiago_pro_head name="head" parent="head_base_link" use_sim_time="$(arg use_sim_time)"/>
+  <xacro:tiago_pro_head name="head" parent="head_base_link" use_sim_time="$(arg use_sim_time)" camera_model="$(arg camera_model)"/>
 </robot>

File: tiago_pro_head_description/urdf/head.urdf.xacro (robot description, xacro)
@@ -26,5 +26,5 @@
   <xacro:property name="head_2_upper_limit" value="0.34907"/>
   <xacro:property name="head_eps" value="${0.07}" />
-  <xacro:macro name="tiago_pro_head" params="name parent use_sim_time:=^|false">
+  <xacro:macro name="tiago_pro_head" params="name parent camera_model use_sim_time:=^|false">
     <!-- Head Link 1-->
     <link name="${name}_1_link">
@@ -117,8 +117,11 @@
       <implicitSpringDamper>1</implicitSpringDamper>
     </gazebo>
+    <!-- Cameras-->
     <!-- Head camera:Intel D435 -->
-    <xacro:sensor_d435 parent="${name}_2_link" name="${name}_front_camera" topics_ns="${name}_front_camera" use_nominal_extrinsics="${use_sim_time}">
-      <origin xyz="-0.0416 0.1555 0" rpy="1.5708 0 3.1416" />
-    </xacro:sensor_d435>
+    <xacro:if value="${camera_model == 'realsense-d435'}">
+      <xacro:sensor_d435 parent="${name}_2_link" name="${name}_front_camera" topics_ns="${name}_front_camera" use_nominal_extrinsics="${use_sim_time}">
+        <origin xyz="-0.0416 0.1555 0" rpy="1.5708 0 3.1416" />
+      </xacro:sensor_d435>
+    </xacro:if>
   </xacro:macro>
   <!-- EYE FRAMES -->

Commit message: Remove unecessary link + fix base_link inertia + update collision meshes + add new head_base_link meshes

File: tiago_pro_head_description/robots/tiago_pro_head.urdf.xacro (robot description, xacro)
@@ -23,6 +23,35 @@
   <xacro:include filename="$(find tiago_pro_head_description)/ros2_control/ros2_control.urdf.xacro" />
   <xacro:tiago_pro_head_ros2_control/>
-  <xacro:include filename="$(find tiago_pro_head_description)/urdf/head_base.urdf.xacro" />
-  <xacro:tiago_pro_head_base/>
+  <link name="world"/>
+  <joint name="head_base_joint" type="fixed">
+      <origin xyz="0 0 1.0" rpy="0 0 0" />
+      <parent link="world" />
+      <child link="head_base_link" />
+  </joint>
+  <link name="head_base_link">
+    <inertial>
+      <origin xyz="-0.01043 0.03314 -0.07485" rpy="0 0 0" />
+      <mass value="2.86228" />
+      <inertia ixx="0.02768" ixy="-0.00010" ixz="-0.00007"
+          iyy="0.01744" iyz="0.00170"
+          izz="0.03518" />
+    </inertial>
+    <visual>
+        <origin xyz="0 0 -0.13584" rpy="0 0 0" />
+        <geometry>
+            <mesh filename="package://tiago_pro_head_description/meshes/head_base_link.stl" />
+        </geometry>
+        <material name="">
+            <color rgba="1 1 1 1" />
+        </material>
+    </visual>
+    <collision>
+      <origin xyz="0 0 -0.13584" rpy="0 0 0" />
+      <geometry>
+          <mesh
+          filename="package://tiago_pro_head_description/meshes/head_base_link_collision.stl" />
+      </geometry>
+    </collision>
+  </link>
   <xacro:tiago_pro_head name="head" parent="head_base_link" use_sim_time="$(arg use_sim_time)" camera_model="$(arg camera_model)"/>
 </robot>

Commit message: Fix screen link + base_link + update link_2 position stl

File: tiago_pro_head_description/robots/tiago_pro_head.urdf.xacro (robot description, xacro)
@@ -25,6 +25,12 @@
   <link name="world"/>
   <joint name="head_base_joint" type="fixed">
-      <origin xyz="0 0 1.0" rpy="0 0 0" />
+      <origin xyz="0 0 0" rpy="0 0 0" />
       <parent link="world" />
+      <child link="base_link" />
+  </joint>
+  <link name="base_link"/>
+  <joint name="base_joint" type="fixed">
+      <origin xyz="0 0 0.137868" rpy="0 0 0" />
+      <parent link="base_link" />
       <child link="head_base_link" />
   </joint>
@@ -38,5 +44,5 @@
     </inertial>
     <visual>
-        <origin xyz="0 0 -0.13584" rpy="0 0 0" />
+        <origin xyz="0 0 -0.137868" rpy="0 0 0" />
         <geometry>
             <mesh filename="package://tiago_pro_head_description/meshes/head_base_link.stl" />
@@ -47,5 +53,5 @@
     </visual>
     <collision>
-      <origin xyz="0 0 -0.13584" rpy="0 0 0" />
+      <origin xyz="0 0 -0.137868" rpy="0 0 0" />
       <geometry>
           <mesh

File: tiago_pro_head_description/urdf/head.urdf.xacro (robot description, xacro)
@@ -97,8 +97,11 @@
     <link name="${name}_screen_link">
       <visual>
-        <origin rpy="${90.0 * deg_to_rad} 0 ${-90.0 * deg_to_rad}" xyz="-0.105 0 0"/>
+        <origin rpy="${90.0 * deg_to_rad} 0 ${-90.0 * deg_to_rad}" xyz="0 0 0"/>
         <geometry>
           <box size="0.17282 0.10824 0.005"/>
         </geometry>
+        <material name="">
+          <color rgba="0 0 0 1" />
+        </material>
       </visual>
     </link>
@@ -120,5 +123,5 @@
       <parent link="${name}_2_link" />
       <child link="${name}_screen_link" />
-      <origin xyz="0.0528 0.08 0.0" rpy="${-90.0 * deg_to_rad} 0 0" />
+      <origin xyz="-0.05584 0.083935 0.0" rpy="${-90.0 * deg_to_rad} 0 0" />
     </joint>
     <gazebo reference="${name}_1_link">

Commit message: Fix head_2_link oriontation

File: tiago_pro_head_description/robots/tiago_pro_head.urdf.xacro (robot description, xacro)
@@ -26,4 +26,5 @@
   <joint name="head_base_joint" type="fixed">
       <origin xyz="0 0 0" rpy="0 0 0" />
+      <!-- <origin xyz="2.40654 -3.4 0.659997" rpy="0 0 ${-90 * deg_to_rad}" /> -->
       <parent link="world" />
       <child link="base_link" />

File: tiago_pro_head_description/urdf/head.urdf.xacro (robot description, xacro)
@@ -64,9 +64,9 @@
     <link name="${name}_2_link">
       <inertial>
-        <origin xyz="-0.00875103486217405 0.114127350051331 -0.000389070804431699"  rpy="0 0 0" />
-        <mass value="0.846359357446667" />
-        <inertia ixx="0.00623850186261437" ixy="-0.000550112126953165" ixz="-9.403405403969E-06"
-          iyy="0.0050320204467172" iyz="-5.68886635279132E-06"
-          izz="0.0024981099013485" />
+        <origin xyz="0.01201 -0.10656 -0.00075"  rpy="0 0 0" />
+        <mass value="1.32153" />
+        <inertia ixx="0.01065" ixy="-0.00119" ixz="0.00001"
+          iyy="0.00878" iyz="-0.00003"
+          izz="0.00627" />
       </inertial>
       <visual>
@@ -87,5 +87,5 @@
     </link>
     <joint name="head_2_joint" type="revolute">
-      <origin xyz="0.0425 0 0.10585" rpy="1.5708 0 -3.1416" />
+      <origin xyz="0.0425 0 0.10585" rpy="-1.5708 0 0" />
       <parent link="${name}_1_link" />
       <child link="${name}_2_link" />
@@ -97,5 +97,5 @@
     <link name="${name}_screen_link">
       <visual>
-        <origin rpy="${90.0 * deg_to_rad} 0 ${-90.0 * deg_to_rad}" xyz="0 0 0"/>
+        <origin rpy="${90.0 * deg_to_rad} 0 ${90.0 * deg_to_rad}" xyz="0 0 0"/>
         <geometry>
           <box size="0.17282 0.10824 0.005"/>
@@ -123,5 +123,5 @@
       <parent link="${name}_2_link" />
       <child link="${name}_screen_link" />
-      <origin xyz="-0.05584 0.083935 0.0" rpy="${-90.0 * deg_to_rad} 0 0" />
+      <origin xyz="0.05584 -0.083935 0.0" rpy="1.5708 0 0" />
     </joint>
     <gazebo reference="${name}_1_link">
@@ -145,5 +145,5 @@
     <xacro:if value="${camera_model == 'realsense-d435'}">
       <xacro:sensor_d435 parent="${name}_2_link" name="${name}_front_camera" topics_ns="${name}_front_camera" use_nominal_extrinsics="${use_sim_time}">
-        <origin xyz="-0.0416 0.1555 0" rpy="1.5708 0 3.1416" />
+        <origin xyz="0.0416 -0.1555 0" rpy="1.5708 0 0" />
       </xacro:sensor_d435>
     </xacro:if>
@@ -152,5 +152,5 @@
   <link name="sellion_link"/>
   <joint name="sellion_joint" type="fixed">
-    <origin xyz="-0.04 0.09205 0" rpy="${-90 * deg_to_rad} ${180 * deg_to_rad} 0"/>
+    <origin xyz="0.04 -0.09205 0" rpy="1.5708 0 0"/>
     <child link="sellion_link" />
     <parent link="head_2_link"/>

Commit message: Update tiago_pro_head.urdf.xacro

File: tiago_pro_head_description/robots/tiago_pro_head.urdf.xacro (robot description, xacro)
@@ -26,5 +26,4 @@
   <joint name="head_base_joint" type="fixed">
       <origin xyz="0 0 0" rpy="0 0 0" />
-      <!-- <origin xyz="2.40654 -3.4 0.659997" rpy="0 0 ${-90 * deg_to_rad}" /> -->
       <parent link="world" />
       <child link="base_link" />

Commit message: remove realsense overlay

File: tiago_pro_head_description/robots/tiago_pro_head.urdf.xacro (robot description, xacro)
@@ -17,7 +17,9 @@
   <xacro:arg name="use_sim_time" default="false"/>
   <xacro:arg name="is_public_sim" default="false"/>
+  <xacro:arg name="namespace" default=""/>
   <xacro:property name="camera_model" value="$(arg camera_model)" />
   <xacro:property name="use_sim_time" value="$(arg use_sim_time)" />
   <xacro:property name="is_public_sim" value="$(arg is_public_sim)" />
+  <xacro:property name="namespace" value="$(arg namespace)" />
     <!-- ROS 2 Control -->
   <xacro:include filename="$(find tiago_pro_head_description)/ros2_control/ros2_control.urdf.xacro" />

File: tiago_pro_head_description/urdf/head.urdf.xacro (robot description, xacro)
@@ -14,6 +14,6 @@
 <robot xmlns:xacro="http://ros.org/wiki/xacro">
   <!--File includes-->
-  <xacro:include filename="$(find realsense2_description)/urdf/_d435.urdf.xacro" />
-  <xacro:include filename="$(find realsense2_description)/urdf/_d455.urdf.xacro" />
+  <xacro:include filename="$(find pal_urdf_utils)/urdf/camera/realsense_d435.urdf.xacro" />
+  <xacro:include filename="$(find pal_urdf_utils)/urdf/camera/realsense_d455.urdf.xacro" />
   <!-- Tools -->
   <xacro:include filename="$(find pal_urdf_utils)/urdf/deg_to_rad.urdf.xacro" />
@@ -154,13 +154,13 @@
     <!-- Head camera:Intel D435 -->
     <xacro:if value="${camera_model == 'realsense-d435'}">
-      <xacro:sensor_d435 parent="${name}_2_link" name="${name}_front_camera" topics_ns="${name}_front_camera" use_nominal_extrinsics="${use_sim_time}">
+      <xacro:realsense_d435 parent="${name}_2_link" name="${name}_front_camera" use_nominal_extrinsics="${use_sim_time}">
         <origin xyz="0.0416 -0.1555 0" rpy="1.5708 0 0" />
-      </xacro:sensor_d435>
+      </xacro:realsense_d435>
     </xacro:if>
     <!-- Head camera:Intel D455 -->
     <xacro:if value="${camera_model == 'realsense-d455'}">
-      <xacro:sensor_d455 parent="${name}_2_link" name="${name}_front_camera" topics_ns="${name}_front_camera" use_nominal_extrinsics="${use_sim_time}">
+      <xacro:realsense_d455 parent="${name}_2_link" name="${name}_front_camera" use_nominal_extrinsics="${use_sim_time}">
         <origin xyz="0.040453 -0.1565 0" rpy="1.5708 0 0" />
-      </xacro:sensor_d455>
+      </xacro:realsense_d455>
     </xacro:if>
   </xacro:macro>

Commit message: added mujoco description

File: tiago_pro_head_description/robots/tiago_pro_head.urdf.xacro (robot description, xacro)
@@ -19,8 +19,17 @@
   <xacro:arg name="namespace" default=""/>
   <xacro:arg name="gazebo_version" default="classic"/>
+  <!-- mujoco-ros2-control, mujoco, gazebo, no-simulation -->
+  <xacro:arg name="sim_type" default="gazebo" />
+  <!-- false, position, motor -->
+  <xacro:arg name="mj_control" default="false" />
+  <xacro:arg name="world_name" default="floor" />
   <xacro:property name="camera_model" value="$(arg camera_model)" />
   <xacro:property name="use_sim_time" value="$(arg use_sim_time)" />
   <xacro:property name="is_public_sim" value="$(arg is_public_sim)" />
   <xacro:property name="namespace" value="$(arg namespace)" />
+  <!-- Mujoco properties -->
+  <xacro:property name="sim_type" value="$(arg sim_type)" />
+  <xacro:property name="mj_control" value="$(arg mj_control)"/>
+  <xacro:property name="world_name" value="$(arg world_name)"/>
   <xacro:property name="gazebo_version" value="$(arg gazebo_version)" />
     <!-- ROS 2 Control -->
@@ -65,3 +74,39 @@
   </link>
   <xacro:tiago_pro_head name="head" parent="head_base_link" use_sim_time="$(arg use_sim_time)" camera_model="$(arg camera_model)"/>
+  <xacro:if value="${sim_type in ['mujoco', 'mujoco-ros2-control']}">
+    <xacro:include filename="$(find tiago_pro_head_description)/mujoco/mj_tags.xacro" />
+    <xacro:include filename="$(find pal_mujoco_scenes)/scenes/${world_name}.xacro" />
+    <mujoco_inputs>
+      <!-- Mujoco environment -->
+      <raw_inputs>
+      <!-- Actuator-->
+        <xacro:if value="${sim_type == 'mujoco'}">
+          <actuator>
+            <xacro:mj_head_actuators/>
+          </actuator>
+        </xacro:if>
+      </raw_inputs>
+      <processed_inputs>
+        <!-- Specifying decompose_mesh will set the `decompose` flag when using obj2mjcf -->
+        <!-- <decompose_mesh mesh_name="arm2_link" threshold="0.05"/>
+        <decompose_mesh mesh_name="arm3_link" threshold="0.05"/> -->
+        <!-- <decompose_mesh mesh_name="arm4_link" threshold="0.05"/> -->
+        <!-- The camera with the specified values will be added at the specified site name. -->
+        <!-- The position and quaterinion will be filled in by the converter -->
+        <!-- Realsense_d435 -->
+        <camera site="head_front_camera_color_eye_frame" name="head" fovy="42" mode="fixed" resolution="848 480"/>
+        <!-- Adds a lidar tag below a site tag to support a lidar sensor. -->
+        <!-- In the URDF, we assume that that the sensor frame has the Z-axis pointed directly up in the sensor -->
+        <!-- frame. This tag will create rangefinders in the MJCF between min_angle and max_angle at each -->
+        <!-- angle_increment rotated about the replicate frame's Y axis. The hardware intercface then combines -->
+        <!-- them into a single LaserScan message. -->
+        <!-- <lidar ref_site="torso_link" sensor_name="rf" min_angle="-0.3" max_angle="0.3" angle_increment="0.025" /> -->
+        <!-- The element with the type and name as listed below will be modified with the remaining attributes -->
+        <!-- If the attribute already existed, it will be overwritten -->
+        <!-- Note that the type and name elements are required -->
+        <!-- <modify_element type="joint" name="joint1" frictionloss="1.0" damping="2.0"/>
+        <modify_element type="body" name="forearm" gravcomp="1.0"/> -->
+      </processed_inputs>
+    </mujoco_inputs>
+  </xacro:if>
 </robot>

Commit message: added mujoco ros2 control

File: tiago_pro_head_description/robots/tiago_pro_head.urdf.xacro (robot description, xacro)
@@ -95,5 +95,5 @@
         <!-- The position and quaterinion will be filled in by the converter -->
         <!-- Realsense_d435 -->
-        <camera site="head_front_camera_color_eye_frame" name="head" fovy="42" mode="fixed" resolution="848 480"/>
+        <!-- <camera site="head_front_camera_color_eye_frame" name="head" fovy="42" mode="fixed" resolution="848 480"/> -->
         <!-- Adds a lidar tag below a site tag to support a lidar sensor. -->
         <!-- In the URDF, we assume that that the sensor frame has the Z-axis pointed directly up in the sensor -->

File: tiago_pro_head_description/ros2_control/ros2_control.urdf.xacro (robot description, xacro)
@@ -13,10 +13,10 @@
  -->
 <robot xmlns:xacro="http://ros.org/wiki/xacro" name="tiago_pro_head" >
-    <xacro:macro name="tiago_pro_head_ros2_control" params="use_sim_time:=^|false">
+  <xacro:macro name="tiago_pro_head_ros2_control" params="use_sim_time:=^|false">
     <xacro:include filename="$(find tiago_pro_head_description)/urdf/head.ros2_control.xacro" />
-    <xacro:unless value="$(arg use_sim_time)">
-      <ros2_control name="ros2_control_tiago_pro_head_system" type="system">
-          <hardware>
-            <xacro:if value="${use_sim_time}">
+    <ros2_control name="ros2_control_tiago_pro_head_system" type="system">
+        <hardware>
+          <xacro:if value="${use_sim_time}">
+            <xacro:if value="${sim_type == 'gazebo'}">
               <xacro:if value="${gazebo_version == 'classic'}">
                 <plugin>gazebo_ros2_control/GazeboSystem</plugin>
@@ -26,22 +26,31 @@
               </xacro:if>
             </xacro:if>
-            <xacro:unless value="${use_sim_time}">
-              <plugin>robot_control/RobotControl</plugin>
-            </xacro:unless>
-          </hardware>
-        <xacro:ros2_control_head />
-      </ros2_control>
-    </xacro:unless>
-    <xacro:if value="${gazebo_version == 'classic'}">
-      <plugin filename="libgazebo_ros2_control.so" name="gazebo_ros2_control">
-        <parameters>$(find tiago_pro_head_description)/ros2_control/gazebo_controller_manager_cfg.yaml</parameters>
-      </plugin>
-    </xacro:if>
-    <xacro:if value="${gazebo_version == 'gazebo'}">
-      <plugin filename="gz_ros2_control-system" name="gz_ros2_control::GazeboSimROS2ControlPlugin">
-        <robot_param>robot_description</robot_param>
-        <robot_param_node>robot_state_publisher</robot_param_node>
-        <parameters>$(find tiago_pro_head_description)/ros2_control/gazebo_controller_manager_cfg.yaml</parameters>
-      </plugin>
+            <xacro:if value="${sim_type == 'mujoco-ros2-control'}">
+              <plugin>mujoco_ros2_control/MujocoSystemInterface</plugin>
+              <!-- Override the slowdown settings in the Simulate App and run at 3x speed -->
+              <param name="sim_speed_factor">1.0</param>
+            </xacro:if>
+          </xacro:if>
+          <xacro:unless value="${use_sim_time}">
+            <plugin>robot_control/RobotControl</plugin>
+          </xacro:unless>
+        </hardware>
+        <xacro:ros2_control_head sim_type="${sim_type}"/>
+    </ros2_control>
+    <xacro:if value="${use_sim_time}">
+      <xacro:if value="${sim_type == 'gazebo'}">
+        <xacro:if value="${gazebo_version == 'classic'}">
+          <plugin filename="libgazebo_ros2_control.so" name="gazebo_ros2_control">
+            <parameters>$(find tiago_pro_head_description)/ros2_control/gazebo_controller_manager_cfg.yaml</parameters>
+          </plugin>
+        </xacro:if>
+        <xacro:if value="${gazebo_version == 'gazebo'}">
+          <plugin filename="gz_ros2_control-system" name="gz_ros2_control::GazeboSimROS2ControlPlugin">
+            <robot_param>robot_description</robot_param>
+            <robot_param_node>robot_state_publisher</robot_param_node>
+            <parameters>$(find tiago_pro_head_description)/ros2_control/gazebo_controller_manager_cfg.yaml</parameters>
+          </plugin>
+        </xacro:if>
+      </xacro:if>
     </xacro:if>
   </xacro:macro>

File: tiago_pro_head_description/urdf/head.ros2_control.xacro (robot description, xacro)
@@ -14,9 +14,9 @@
 <robot xmlns:xacro="http://ros.org/wiki/xacro">
   <!-- ROS 2 Control -->
-  <xacro:macro name="ros2_control_head" >
-    <xacro:ros2_control_head_joint name="head_1" reduction="1.0" offset_value="0.0" />
-    <xacro:ros2_control_head_joint name="head_2" reduction="1.0" offset_value="0.0" />
+  <xacro:macro name="ros2_control_head" params="sim_type:=gazebo">
+    <xacro:ros2_control_head_joint name="head_1" reduction="1.0" offset_value="0.0" sim_type="${sim_type}" />
+    <xacro:ros2_control_head_joint name="head_2" reduction="1.0" offset_value="0.0" sim_type="${sim_type}"/>
   </xacro:macro>
-  <xacro:macro name="ros2_control_head_joint" params="name reduction offset_value" >
+  <xacro:macro name="ros2_control_head_joint" params="name reduction offset_value sim_type:=gazebo" >
     <joint name="${name}_joint">
       <command_interface name="position" />
@@ -25,6 +25,8 @@
       <state_interface name="effort" />
     </joint>
-    <xacro:include filename="$(find tiago_pro_head_description)/urdf/head.transmission.urdf.xacro" />
-    <xacro:head_transmission name="${name}" reduction="1" offset_value="${offset_value}" />
+    <xacro:if value="${sim_type != 'mujoco-ros2-control'}">
+      <xacro:include filename="$(find tiago_pro_head_description)/urdf/head.transmission.urdf.xacro" />
+      <xacro:head_transmission name="${name}" reduction="1" offset_value="${offset_value}" />
+    </xacro:if>
   </xacro:macro>
 </robot>
