Commit message: move mj_tags to the head.urdf.xacro

File: tiago_pro_head_description/robots/tiago_pro_head.urdf.xacro (robot description, xacro)
@@ -75,38 +75,5 @@
   <xacro:tiago_pro_head name="head" parent="head_base_link" use_sim_time="$(arg use_sim_time)" camera_model="$(arg camera_model)"/>
   <xacro:if value="${sim_type in ['mujoco', 'mujoco-ros2-control']}">
-    <xacro:include filename="$(find tiago_pro_head_description)/mujoco/mj_tags.xacro" />
-    <xacro:include filename="$(find pal_mujoco_scenes)/scenes/${world_name}.xacro" />
-    <mujoco_inputs>
-      <!-- Mujoco environment -->
-      <raw_inputs>
-      <!-- Actuator-->
-        <xacro:if value="${sim_type == 'mujoco'}">
-          <actuator>
-            <xacro:mj_head_actuators/>
-          </actuator>
-        </xacro:if>
-      </raw_inputs>
-      <processed_inputs>
-        <!-- Specifying decompose_mesh will set the `decompose` flag when using obj2mjcf -->
-        <!-- <decompose_mesh mesh_name="arm2_link" threshold="0.05"/>
-        <decompose_mesh mesh_name="arm3_link" threshold="0.05"/> -->
-        <!-- <decompose_mesh mesh_name="arm4_link" threshold="0.05"/> -->
-        <!-- The camera with the specified values will be added at the specified site name. -->
-        <!-- The position and quaterinion will be filled in by the converter -->
-        <!-- Realsense_d435 -->
-        <!-- <camera site="head_front_camera_color_eye_frame" name="head" fovy="42" mode="fixed" resolution="848 480"/> -->
-        <!-- Adds a lidar tag below a site tag to support a lidar sensor. -->
-        <!-- In the URDF, we assume that that the sensor frame has the Z-axis pointed directly up in the sensor -->
-        <!-- frame. This tag will create rangefinders in the MJCF between min_angle and max_angle at each -->
-        <!-- angle_increment rotated about the replicate frame's Y axis. The hardware intercface then combines -->
-        <!-- them into a single LaserScan message. -->
-        <!-- <lidar ref_site="torso_link" sensor_name="rf" min_angle="-0.3" max_angle="0.3" angle_increment="0.025" /> -->
-        <!-- The element with the type and name as listed below will be modified with the remaining attributes -->
-        <!-- If the attribute already existed, it will be overwritten -->
-        <!-- Note that the type and name elements are required -->
-        <!-- <modify_element type="joint" name="joint1" frictionloss="1.0" damping="2.0"/>
-        <modify_element type="body" name="forearm" gravcomp="1.0"/> -->
-      </processed_inputs>
-    </mujoco_inputs>
+    <xacro:tiago_pro_head_mj world_name="${world_name}" mj_control="${mj_control}"/>
   </xacro:if>
 </robot>

File: tiago_pro_head_description/urdf/head.urdf.xacro (robot description, xacro)
@@ -174,4 +174,38 @@
     </xacro:if>
   </xacro:macro>
+  <xacro:macro name="tiago_pro_head_mj" params="mj_control world">
+    <xacro:include filename="$(find tiago_pro_head_description)/mujoco/mj_tags.xacro" />
+    <xacro:include filename="$(find pal_mujoco_scenes)/scenes/${world_name}.xacro" />
+    <mujoco_inputs>
+      <!-- Mujoco environment -->
+      <scene>
+        <xacro:mj_scene/>
+      </scene>
+      <raw_inputs>
+        <!-- Actuator-->
+        <actuator>
+          <xacro:mj_head_actuators mj_control="${mj_control}"/>
+        </actuator>
+      </raw_inputs>
+      <processed_inputs>
+        <!-- Specifying decompose_mesh will set the `decompose` flag when using obj2mjcf -->
+        <!-- <decompose_mesh mesh_name="{mesh_name}" threshold=" {threshold_value}"/> -->
+        <!-- The camera with the specified values will be added at the specified site name. -->
+        <!-- The position and quaterinion will be filled in by the converter -->
+        <!-- Realsense_d435 -->
+        <camera site="head_front_camera_color_eye_frame" name="head" fovy="42" mode="fixed" resolution="848 480"/>
+        <!-- Adds a lidar tag below a site tag to support a lidar sensor. -->
+        <!-- In the URDF, we assume that that the sensor frame has the Z-axis pointed directly up in the sensor -->
+        <!-- frame. This tag will create rangefinders in the MJCF between min_angle and max_angle at each -->
+        <!-- angle_increment rotated about the replicate frame's Y axis. The hardware intercface then combines -->
+        <!-- them into a single LaserScan message. -->
+        <!-- <lidar ref_site="{link_name}" sensor_name="{sensor_name}" min_angle="{min_angle_value}" max_angle="{max_angle_value}" angle_increment="{angle_increment_value}" /> -->
+        <!-- The element with the type and name as listed below will be modified with the remaining attributes -->
+        <!-- If the attribute already existed, it will be overwritten -->
+        <!-- Note that the type and name elements are required -->
+        <!-- <modify_element type="{element_type}" name="{element_name}" frictionloss="{value}" damping="{value}"/> -->
+      </processed_inputs>
+    </mujoco_inputs>
+  </xacro:macro>
   <!-- EYE FRAMES -->
   <link name="sellion_link"/>

Commit message: pass sim_type argument as xacro parameter

File: tiago_pro_head_description/robots/tiago_pro_head.urdf.xacro (robot description, xacro)
@@ -19,8 +19,9 @@
   <xacro:arg name="namespace" default=""/>
   <xacro:arg name="gazebo_version" default="classic"/>
-  <!-- mujoco-ros2-control, mujoco, gazebo, no-simulation -->
+  <!-- mujoco-ros2-control, mujoco, gazebo-->
   <xacro:arg name="sim_type" default="gazebo" />
   <!-- false, position, motor -->
   <xacro:arg name="mj_control" default="false" />
+  <!-- floor -->
   <xacro:arg name="world_name" default="floor" />
   <xacro:property name="camera_model" value="$(arg camera_model)" />
@@ -33,7 +34,7 @@
   <xacro:property name="world_name" value="$(arg world_name)"/>
   <xacro:property name="gazebo_version" value="$(arg gazebo_version)" />
-    <!-- ROS 2 Control -->
+  <!-- ROS 2 Control -->
   <xacro:include filename="$(find tiago_pro_head_description)/ros2_control/ros2_control.urdf.xacro" />
-  <xacro:tiago_pro_head_ros2_control/>
+  <xacro:tiago_pro_head_ros2_control use_sim_time="${use_sim_time}" sim_type="${sim_type}"/>
   <link name="world"/>
   <joint name="head_base_joint" type="fixed">

File: tiago_pro_head_description/urdf/head.ros2_control.xacro (robot description, xacro)
@@ -14,9 +14,9 @@
 <robot xmlns:xacro="http://ros.org/wiki/xacro">
   <!-- ROS 2 Control -->
-  <xacro:macro name="ros2_control_head" params="sim_type:=gazebo">
+  <xacro:macro name="ros2_control_head" params="sim_type:=^|gazebo">
     <xacro:ros2_control_head_joint name="head_1" reduction="1.0" offset_value="0.0" sim_type="${sim_type}" />
     <xacro:ros2_control_head_joint name="head_2" reduction="1.0" offset_value="0.0" sim_type="${sim_type}"/>
   </xacro:macro>
-  <xacro:macro name="ros2_control_head_joint" params="name reduction offset_value sim_type:=gazebo" >
+  <xacro:macro name="ros2_control_head_joint" params="name reduction offset_value sim_type:=^|gazebo" >
     <joint name="${name}_joint">
       <command_interface name="position" />

File: tiago_pro_head_description/urdf/head.urdf.xacro (robot description, xacro)
@@ -13,4 +13,5 @@
 -->
 <robot xmlns:xacro="http://ros.org/wiki/xacro">
+  <xacro:macro name="tiago_pro_head" params="name parent camera_model use_sim_time:=^|false">
   <!--File includes-->
   <xacro:include filename="$(find pal_urdf_utils)/urdf/camera/realsense_d435.urdf.xacro" />

Commit message: add check for the values of the sim_type argument

File: tiago_pro_head_description/robots/tiago_pro_head.urdf.xacro (robot description, xacro)
@@ -34,4 +34,11 @@
   <xacro:property name="world_name" value="$(arg world_name)"/>
   <xacro:property name="gazebo_version" value="$(arg gazebo_version)" />
+  <!-- Properties check -->
+  <xacro:if value="${sim_type not in ['mujoco-ros2-control', 'mujoco', 'gazebo']}">
+    <xacro:wrong_sim_type />
+  </xacro:if>
+  <xacro:unless value="$(arg use_sim_time)">
+    <xacro:property name="sim_type" value="gazebo" />
+  </xacro:unless>
   <!-- ROS 2 Control -->
   <xacro:if value="${sim_type != 'mujoco'}">
